File: Starforge Basic/Hardware/PCB/_restore_backup_2026-09-14T19-05-20-038/PCB.kicad_sch (KiCad schematic)
At the start: 74 parts, among them CN1 XT30UPB-M, CN2 2060-453-HDGC, CN3 2060-452-HDGC, CN4 2060-453-HDGC, CN6 2060-453-HDGC, CN7 2060-453-HDGC, J1 Connector, USB-TYPE-C-16P, SW1 TS-1187A-B-A-B, U1 RP2350B_C42415655, U3 BMP581, U4 ICM-45686, U5 BQ25883RGER, U6 LMR51430YFDDCR, U7 TPS630701RNMR, U8 GD25Q128ESIGR, X2 X322512MSB4SI

Commit message: base
Parts:
- removed C26, C27: CL21A106KAYNNNE, easyeda2kicad:C0805, symbol easyeda2kicad:CL21A106KAYNNNE
- removed C28, C29: 470 uF, Capacitor_SMD:CP_Elec_8x10.5, symbol Device:C_Polarized
- removed R19: 0402WGF1001TCE, easyeda2kicad:R0402, symbol easyeda2kicad:0402WGF1001TCE
- removed R20, R21: 0402WGF4701TCE, easyeda2kicad:R0402, symbol easyeda2kicad:0402WGF4701TCE
- removed SW1: TS-1187A-B-A-B, easyeda2kicad:SW-SMD_4P-L5.1-W5.1-P3.70-LS6.5-TL_H1.5, symbol easyeda2kicad:TS-1187A-B-A-B
Connections:
- net +3V3: now also U3.6 (CSB)
- net GND: no longer C23.1
- net at C24.1, CN4.2, CN6.2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: now also C23.1; no longer C23.2, U7.5 (FB), U7.7 (VOUT), U7.8 (VOUT)
- net at CN6.1: no longer U1.23 (GPIO23)
- net at CN4.1: no longer U1.22 (GPIO22)
- net at U1.7 (GPIO9): no longer U3.6 (CSB)
- net at CN2.1: no longer U1.21 (GPIO21)
- net at CN7.1: no longer U1.25 (GPIO24)
- new net: C23.2, U7.5 (FB), U7.7 (VOUT), U7.8 (VOUT)
