File: Hardware/PCB/PCB.kicad_sch (KiCad schematic)
At the start: 40 parts, among them CN1 XT30UPB-M, U1 BQ25883RGER, U3 TPS82130SILR, U4 TPS82130SILR

Commit message: Power IC complete
Parts:
- added Card1: TF-01A, easyeda2kicad:TF-SMD_TF-01A, symbol OG FCFILE:TF-01A
Connections:
- net +3.3V: no longer C13.2, R15.2, R16.2, U4.4 (VOUT), U4.5 (VOUT)
- net PG3v3: no longer R15.1, U4.7 (PG)
- new net +5V: C13.2, R15.2, R16.2, U4.4 (VOUT), U4.5 (VOUT)
- new net PG5V: R15.1, U4.7 (PG)
Changed lines of the file:
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@@
 	)
 	(rectangle
+		(start 74.295 102.87)
+		(end 148.59 170.18)
+		(stroke
+			(width 0)
+			(type default)
+		)
+		(fill
+			(type none)
+		)
+	)
+	(rectangle
 		(start 19.05 143.51)
 		(end 71.755 184.15)
@@
 	(text "Battery charger/input"
 		(exclude_from_sim no)
-		(at 107.188 97.282 0)
+		(at 103.886 99.314 0)
 		(effects
 			(font
@@
 		)
 	)
-	(label "PG3v3"
+	(label "PG5V"
 		(at 20.32 170.18 0)
 		(effects
@@
 		)
 	)
-	(label "PG3v3"
+	(label "PG5V"
 		(at 62.23 158.75 180)
 		(effects
@@
 	)
 	(symbol
-		(lib_id "power:+3.3V")
-		(at 66.04 170.18 0)
+		(lib_id "Device:R_Small")
+		(at 64.77 161.29 90)
 		(unit 1)
 		(body_style 1)
@@
 		(in_pos_files yes)
 		(dnp no)
-		(property "Reference" "#PWR036"
-			(at 66.04 173.99 0)
-			(hide yes)
+		(property "Reference" "R17"
+			(at 64.77 157.48 90)
 			(show_name no)
 			(do_not_autoplace no)
 			(effects
 				(font
-					(size 1.27 1.27)
+					(size 1.016 1.016)
 				)
 			)
 		)
-		(property "Value" "+3.3V"
-			(at 66.04 166.624 0)
+		(property "Value" "20K"
+			(at 64.77 159.258 90)
 			(show_name no)
 			(do_not_autoplace no)
@@
 		)
 		(property "Footprint" ""
-			(at 66.04 170.18 0)
+			(at 64.77 161.29 0)
 			(hide yes)
 			(show_name no)
@@
 		)
 		(property "Datasheet" ""
-			(at 66.04 170.18 0)
+			(at 64.77 161.29 0)
 			(hide yes)
 			(show_name no)
@@
 			)
 		)
-		(property "Description" "Power symbol creates a global label with name \"+3.3V\""
-			(at 66.04 170.18 0)
+		(property "Description" "Resistor, small symbol"
+			(at 64.77 161.29 0)
 			(hide yes)
 			(show_name no)
@@
 		(pin "1"
 		)
+		(pin "2"
+		)
 		(instances
 			(project "PCB"
 				(path "/baf65b9d-8965-47ba-bcd0-4660d1815206"
-					(reference "#PWR036")
+					(reference "R17")
 					(unit 1)
 				)
@@
 	)
 	(symbol
-		(lib_id "Device:R_Small")
-		(at 64.77 161.29 90)
+		(lib_id "power:GND")
+		(at 118.11 66.04 0)
+		(mirror y)
 		(unit 1)
 		(body_style 1)
@@
 		(in_pos_files yes)
 		(dnp no)
-		(property "Reference" "R17"
-			(at 64.77 157.48 90)
+		(property "Reference" "#PWR014"
+			(at 118.11 72.39 0)
+			(hide yes)
 			(show_name no)
 			(do_not_autoplace no)
 			(effects
 				(font
-					(size 1.016 1.016)
+					(size 1.27 1.27)
 				)
 			)
 		)
-		(property "Value" "20K"
-			(at 64.77 159.258 90)
+		(property "Value" "GND"
+			(at 118.11 69.85 0)
 			(show_name no)
 			(do_not_autoplace no)
@@
 		)
 		(property "Footprint" ""
-			(at 64.77 161.29 0)
+			(at 118.11 66.04 0)
 			(hide yes)
 			(show_name no)
@@
 		)
 		(property "Datasheet" ""
-			(at 64.77 161.29 0)
+			(at 118.11 66.04 0)
 			(hide yes)
 			(show_name no)
@@
 			)
 		)
-		(property "Description" "Resistor, small symbol"
-			(at 64.77 161.29 0)
+		(property "Description" "Power symbol creates a global label with name \"GND\" , ground"
+			(at 118.11 66.04 0)
 			(hide yes)
 			(show_name no)
@@
 		(pin "1"
 		)
-		(pin "2"
-		)
 		(instances
 			(project "PCB"
 				(path "/baf65b9d-8965-47ba-bcd0-4660d1815206"
-					(reference "R17")
+					(reference "#PWR014")
 					(unit 1)
 				)
@@
 	(symbol
 		(lib_id "power:GND")
-		(at 118.11 66.04 0)
+		(at 96.52 77.47 0)
 		(mirror y)
 		(unit 1)
@@
 		(in_pos_files yes)
 		(dnp no)
-		(property "Reference" "#PWR014"
-			(at 118.11 72.39 0)
+		(property "Reference" "#PWR018"
+			(at 96.52 83.82 0)
 			(hide yes)
 			(show_name no)
@@
 		)
 		(property "Value" "GND"
-			(at 118.11 69.85 0)
+			(at 96.52 81.28 0)
 			(show_name no)
 			(do_not_autoplace no)
@@
 		)
 		(property "Footprint" ""
-			(at 118.11 66.04 0)
+			(at 96.52 77.47 0)
 			(hide yes)
 			(show_name no)
@@
 		)
 		(property "Datasheet" ""
-			(at 118.11 66.04 0)
+			(at 96.52 77.47 0)
 			(hide yes)
 			(show_name no)
@@
 		)
 		(property "Description" "Power symbol creates a global label with name \"GND\" , ground"
-			(at 118.11 66.04 0)
+			(at 96.52 77.47 0)
 			(hide yes)
 			(show_name no)
@@
 			(project "PCB"
 				(path "/baf65b9d-8965-47ba-bcd0-4660d1815206"
-					(reference "#PWR014")
+					(reference "#PWR018")
 					(unit 1)
 				)
@@
 	)
 	(symbol
-		(lib_id "power:GND")
-		(at 96.52 77.47 0)
-		(mirror y)
+		(lib_id "power:+5V")
+		(at 66.04 170.18 0)
 		(unit 1)
 		(body_style 1)
@@
 		(in_pos_files yes)
 		(dnp no)
-		(property "Reference" "#PWR018"
-			(at 96.52 83.82 0)
+		(property "Reference" "#PWR036"
+			(at 66.04 173.99 0)
 			(hide yes)
 			(show_name no)
@@
 			)
 		)
-		(property "Value" "GND"
-			(at 96.52 81.28 0)
+		(property "Value" "+5V"
+			(at 65.786 166.878 0)
 			(show_name no)
 			(do_not_autoplace no)
@@
 		)
 		(property "Footprint" ""
-			(at 96.52 77.47 0)
+			(at 66.04 170.18 0)
 			(hide yes)
 			(show_name no)
@@
 		)
 		(property "Datasheet" ""
-			(at 96.52 77.47 0)
+			(at 66.04 170.18 0)
 			(hide yes)
 			(show_name no)
@@
 			)
 		)
-		(property "Description" "Power symbol creates a global label with name \"GND\" , ground"
-			(at 96.52 77.47 0)
+		(property "Description" "Power symbol creates a global label with name \"+5V\""
+			(at 66.04 170.18 0)
 			(hide yes)
 			(show_name no)
@@
 			(project "PCB"
 				(path "/baf65b9d-8965-47ba-bcd0-4660d1815206"
-					(reference "#PWR018")
+					(reference "#PWR036")
 					(unit 1)
 				)
@@
 					(unit 1)
 				)
+			)
+		)
+	)
+	(symbol
+		(lib_id "OG FCFILE:TF-01A")
+		(at 115.57 134.62 0)
+		(unit 1)
+		(body_style 1)
+		(exclude_from_sim no)
+		(in_bom yes)
+		(on_board yes)
+		(in_pos_files yes)
+		(dnp no)
+		(fields_autoplaced yes)
+		(property "Reference" "Card1"
+			(at 121.5233 119.38 0)
+			(show_name no)
+			(do_not_autoplace no)
+			(effects
+				(font
+					(size 1.27 1.27)
+				)
+				(justify left)
+			)
+		)
+		(property "Value" "TF-01A"
+			(at 121.5233 121.92 0)
+			(show_name no)
+			(do_not_autoplace no)
+			(effects
+				(font
+					(size 1.27 1.27)
+				)
+				(justify left)
+			)
+		)
+		(property "Footprint" "easyeda2kicad:TF-SMD_TF-01A"
+			(at 115.57 160.02 0)
+			(hide yes)
+			(show_name no)
+			(do_not_autoplace no)
+			(effects
+				(font
+					(size 1.27 1.27)
+				)
+			)
+		)
+		(property "Datasheet" "https://lcsc.com/product-detail/Card-Sockets_TF-01A_C91145.html"
+			(at 115.57 162.56 0)
+			(hide yes)
+			(show_name no)
+			(do_not_autoplace no)
+			(effects
+				(font
+					(size 1.27 1.27)
+				)
+			)
+		)
+		(property "Description" ""
+			(at 115.57 134.62 0)
+			(hide yes)
+			(show_name no)
+			(do_not_autoplace no)
+			(effects
+				(font
+					(size 1.27 1.27)
+				)
+			)
+		)
+		(property "Manufacturer" "韩国韩荣"
+			(at 115.57 165.1 0)
+			(hide yes)
+			(show_name no)
+			(do_not_autoplace no)
+			(effects
+				(font
+					(size 1.27 1.27)
+				)
+			)
+		)
+		(property "MPN" "TF-01A"
+			(at 115.57 167.64 0)
+			(hide yes)
+			(show_name no)
+			(do_not_autoplace no)
+			(effects
+				(font
+					(size 1.27 1.27)
+				)
+			)
+		)
+		(property "LCSC Part" "C91145"
+			(at 115.57 170.18 0)
+			(hide yes)
+			(show_name no)
+			(do_not_autoplace no)
+			(effects
+				(font
+					(size 1.27 1.27)
+				)
+			)
+		)
+		(pin "12"
+		)
+		(pin "13"
+		)
+		(pin "6"
+		)
+		(pin "10"
+		)
+		(pin "3"
+		)
+		(pin "2"
+		)
+		(pin "7"
+		)
+		(pin "9"
+		)
+		(pin "4"
+		)
+		(pin "11"
+		)
+		(pin "8"
+		)
+		(pin "1"
+		)
+		(pin "5"
+		)
+		(instances
+			(project "PCB"
+				(path "/baf65b9d-8965-47ba-bcd0-4660d1815206"
+					(reference "Card1")
+					(unit 1)
+				)

Commit message: Restarted Schematic Finished!
Parts:
- removed R7: 10K, symbol Device:R_Small
- added C15, C19, C20, C22, C24, C28, C29, C30, C31, C32, C33, C34, C35, C36: 100nF, symbol Device:C_Small
- added C16, C17, C18: 10uF, symbol Device:C_Small
- added C21: 10nF, symbol Device:C_Small
- added C23: 2.2uF, symbol Device:C_Small
- added C25, C26, C27, C37: 4.7uF, symbol Device:C_Small
- added H1, H2, H3, H4: MountingHole_Pad, symbol Mechanical:MountingHole_Pad
- added H5: SERVOH1, lcsc_footprints:C2937625_HDR-TH_3P-P2_54-V-M_PZ254V-11-03P, symbol FCFILES:PZ254V-11-03P_C2937625
- added H6: SERVOH2, lcsc_footprints:C2937625_HDR-TH_3P-P2_54-V-M_PZ254V-11-03P, symbol FCFILES:PZ254V-11-03P_C2937625
- added H7: SERVON1, lcsc_footprints:C2937625_HDR-TH_3P-P2_54-V-M_PZ254V-11-03P, symbol FCFILES:PZ254V-11-03P_C2937625
- added H8: SERVON2, lcsc_footprints:C2937625_HDR-TH_3P-P2_54-V-M_PZ254V-11-03P, symbol FCFILES:PZ254V-11-03P_C2937625
- added H9: DEBUG, lcsc_footprints:C2937625_HDR-TH_3P-P2_54-V-M_PZ254V-11-03P, symbol FCFILES:PZ254V-11-03P_C2937625
- added L2: 3.3uH, symbol Device:L_Small
- added R18, R19, R20, R21, R22, R23, R24: 10K, symbol Device:R_Small
- added R25, R26: 1K, symbol Device:R_Small
- added R27: 33, symbol Device:R_Small
- added R28, R29: 27, symbol Device:R_Small
- added SW1: TS-1187A-B-A-B, easyeda2kicad:SW-SMD_4P-L5.1-W5.1-P3.70-LS6.5-TL_H1.5, symbol OG FCFILE:TS-1187A-B-A-B
- added U2: RP2354A, lcsc_footprints:C41378174_QFN-60_L7_0-W7_0-P0_40-TL-EP3_4, symbol FCFILES:RP2354A
- added U5: BMP581, easyeda2kicad:LGA-10_L2.0-W2.0-P0.50-TL_BMP581, symbol OG FCFILE:BMP581
- added U6: ICM-42688-P, lcsc_footprints:C1850418_LGA-14_L3_0-W2_5-P0_50-TL, symbol FCFILES:ICM-42688-P
- added U7: Crystal, lcsc_footprints:C20625731_CRYSTAL-SMD_4P-L3_2-W2_5-BL, symbol FCFILES:ABM8-272-T3_C20625731
- C1, C2, C3, C4: footprint (none) -> PCM_JLCPCB:C_0402
- C5, C7, C8: value 20uF -> 10uF
Connections:
- net CE-BC is gone; now on net GND: U1.3 (~{CE})
- net +3.3V: now also Card1.4 (VDD), C15.2, C16.2, C19.2, C20.2, C21.2, C22.1, C23.1, C25.2, C30.2, C31.2, C32.2, C33.2, C34.2, C35.2, C36.2, R18.1, R19.1, R20.1, R21.1, R22.1, R23.2, R24.2, R26.2, R27.2, U2.1 (IOVDD), U2.11 (IOVDD), U2.20 (IOVDD), U2.30 (IOVDD), U2.38 (IOVDD), U2.44 (ADC_AVDD), U2.45 (IOVDD), U2.49 (VREG_VIN), U2.53 (USB_OTP_VDD), U2.54 (QSPI_IOVDD), U5.1 (VDDIO), U5.10 (VDD), U6.5 (VDDIO), U6.8 (VDD)
- net +5V: now also H7.2, H8.2
- net +7.5V: now also C17.2, C18.2, H5.2, H6.2
- net DNCO: now also R29.2, U2.51 (USB_DM); no longer D1.4
- net DPCO: now also R28.2, U2.52 (USB_DP); no longer D1.6
- net GND: now also Card1.10 (GND), Card1.11 (GND), Card1.12 (GND), Card1.13 (GND), Card1.6 (VSS), C15.1, C16.1, C17.1, C18.1, C19.1, C20.1, C21.1, C22.2, C23.2, C24.1, C25.1, C26.2, C27.1, C28.1, C29.1, C30.1, C31.1, C32.1, C33.1, C34.1, C35.1, C36.1, C37.1, H1.1, H2.1, H3.1, H4.1, H5.1, H6.1, H7.1, H8.1, H9.1, SW1.3 (C), SW1.4 (D), U2.47 (VREG_PGND), U2.61 (EP), U5.3 (VSS), U5.8 (VSS), U5.9 (VSS), U6.11 (RESV), U6.6 (GND), U6.7 (RESV), U7.2 (GND), U7.4 (GND)
- net INT-BC: now also U2.4 (GPIO2)
- net SCL-BC: now also U2.3 (GPIO1)
- net SDA-BC: now also U2.2 (GPIO0)
- net at Card1.1 (DAT2(RSV)): now also R18.2
- net SDCS: now reaches Card1.2 (CDDAT3(CS))
- net SDCS: now also R20.2, U2.28 (GPIO17)
- net SDMOSI: now reaches Card1.3 (CMD(DI))
- net SDMOSI: now also R21.2, U2.31 (GPIO19)
- net SDCLK: now reaches Card1.5 (CLK(SCLK))
- net SDCLK: now also R22.2, U2.29 (GPIO18)
- net SDMISO: now reaches Card1.7 (DAT0(D0))
- net SDMISO: now also R23.1, U2.32 (GPIO20)
- net at Card1.8 (DAT1(RSV)): now also R19.2
- net SDCD: now reaches Card1.9 (CD)
- net SDCD: now also R24.1, U2.33 (GPIO21)
- new net: C37.2, R27.1, U2.46 (VREG_AVDD)
- new net: C24.2, R26.1, U2.26 (RUN)
- new net: H9.3, U2.24 (SWCLK)
- new net: H9.2, U2.25 (SWDIO)
- new net: L2.1, U2.48 (VREG_LX)
- new net: R25.1, U2.60 (QSPI_SS)
- new net: D1.4, R29.1
- new net: R25.2, SW1.1 (A), SW1.2 (B)
- new net: D1.6, R28.1
- new net +1V1: C26.1, C27.2, C28.2, C29.2, L2.2, U2.23 (DVDD), U2.39 (DVDD), U2.50 (VREG_FB), U2.6 (DVDD)
- new net AP_CS_IMU: U2.17 (GPIO13), U6.12 (AP_CS)
- new net AP_SCL_IMU: U2.18 (GPIO14), U6.13 (AP_SCL/AP_SCLK)
- new net AP_SDA_IMU: U2.19 (GPIO15), U6.14 (AP_SDA/AP_SDIO/AP_SDI)
- new net AP_SDO_IMU: U2.16 (GPIO12), U6.1 (AP_SDO/AP_AD0)
- new net BMCSB: U2.13 (GPIO9), U2.14 (GPIO10), U5.6 (CSB)
- new net BMINT: U2.8 (GPIO5), U5.7 (INT)
- new net BMSCK: U2.9 (GPIO6), U5.2 (SCK)
- new net BMSDI: U2.10 (GPIO7), U5.4 (SDI)
- new net BMSDO: U2.12 (GPIO8), U5.5 (SDO)
- new net INT2_IMU: U2.27 (GPIO16), U6.9 (INT2/FSYNC/CLKIN)
- new net INT_IMU: U2.15 (GPIO11), U6.4 (INT1/INT)
- new net SH1: H5.3, U2.34 (GPIO22)
- new net SH2: H6.3, U2.35 (GPIO23)
- new net SN1: H7.3, U2.36 (GPIO24)
- new net SN2: H8.3, U2.37 (GPIO25)
- new net XIN: U2.21 (XIN), U7.1
- new net XOUT: U2.22 (XOUT), U7.3
Other:
- note added: "2"
- note added: "Barometer"
- note added: "IMU"
- note added: "MCU + Servo + Debug + Decoupling"
- note added: "MicroSD Storage"
- note added: "Mounting"
- note added: "Sol Mk. 1"
- moved on the sheet: Card1
